File: power.kicad_sch (KiCad schematic)
At the start: 17 parts, among them J16 Conn_02x08_Eurorack, U41 TLV76733

Commit message: rename symbol & footprint libs
Parts:
- J16: footprint MyParts:Eurorack_Full_IDC_Vertical -> BMCV:Eurorack_Full_IDC_Vertical; symbol MySymbols:Conn_02x08_Eurorack -> BMCV:Conn_02x08_Eurorack
- U41: footprint MyParts:HVSSOP-8-1EP_3x3mm_P0.65mm_EP1.57x1.89mm -> BMCV:HVSSOP-8-1EP_3x3mm_P0.65mm_EP1.57x1.89mm; symbol MySymbols:TLV767XX -> BMCV:TLV767XX
Changed lines of the file:
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@@
 	)
 	(symbol
-		(lib_id "MySymbols:TLV767XX")
+		(lib_id "BMCV:TLV767XX")
 		(at 64.77 39.37 0)
 		(unit 1)
@@
 			)
 		)
-		(property "Footprint" "MyParts:HVSSOP-8-1EP_3x3mm_P0.65mm_EP1.57x1.89mm"
+		(property "Footprint" "BMCV:HVSSOP-8-1EP_3x3mm_P0.65mm_EP1.57x1.89mm"
 			(at 64.77 39.37 0)
 			(effects
@@
 	)
 	(symbol
-		(lib_id "MySymbols:Conn_02x08_Eurorack")
+		(lib_id "BMCV:Conn_02x08_Eurorack")
 		(at 142.24 44.45 180)
 		(unit 1)
@@
 			)
 		)
-		(property "Footprint" "MyParts:Eurorack_Full_IDC_Vertical"
+		(property "Footprint" "BMCV:Eurorack_Full_IDC_Vertical"
 			(at 144.018 25.654 0)
 			(effects

Commit message: switches & led data routing
Parts:
- C9: footprint Capacitor_SMD:C_0603_1608Metric -> Capacitor_SMD:C_0402_1005Metric
Changed lines of the file:
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@@
 			)
 		)
-		(property "Footprint" "Capacitor_SMD:C_0603_1608Metric"
+		(property "Footprint" "Capacitor_SMD:C_0402_1005Metric"
 			(at 48.26 96.52 0)
 			(effects

Commit message: alpha
Parts:
- added C96: 10u, Capacitor_SMD:C_0805_2012Metric, symbol Device:C_Small
- added C97, C98: 22u, Capacitor_SMD:C_0805_2012Metric, symbol Device:C_Small
- C10, C16: LCSC Part # (none) -> C15849
- C14, C17: value 1u -> 100n; LCSC Part # (none) -> C15849
- C15: LCSC Part # (none) -> C45783
- C19: value 1u -> 100n; LCSC Part # (none) -> C14663
- C8: LCSC Part # (none) -> C15195
- C9: footprint Capacitor_SMD:C_0402_1005Metric -> Capacitor_SMD:C_0603_1608Metric; LCSC Part # (none) -> C15849
- D1: LCSC Part # (none) -> C2286
- F1: LCSC Part # (none) -> C20801
- FB1, FB2, FB3, FB4: LCSC Part # (none) -> C114780
- J16: LCSC Part # (none) -> C3406; now not fitted
- R4: LCSC Part # (none) -> C11702
- U41: LCSC Part # (none) -> C2873382
Connections:
- net +12V: now also C17.1, C97.2
- net +12V_RAW: no longer C17.1
- net +5V: now also C19.1, C96.2
- net -12V: now also C14.2, C98.2
- net -12V_RAW: no longer C14.2
- net GND: now also C96.1, C97.1, C98.1
- net at F1.2, FB2.2: no longer C19.1
Other:
- moved on the sheet: C14, C17, C19, FB2, FB3, FB4

Commit message: fix & add bom
Parts:
- C14, C17: LCSC Part # C15849 -> C14663
Changed lines of the file:
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@@
 			)
 		)
-		(property "LCSC Part #" "C15849"
+		(property "LCSC Part #" "C14663"
 			(at 234.95 86.36 0)
 			(effects
@@
 			)
 		)
-		(property "LCSC Part #" "C15849"
+		(property "LCSC Part #" "C14663"
 			(at 234.315 62.23 0)
 			(effects

Commit message: update
Changed lines of the file:
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@@
 	)
 	(label "PWR_LED_K"
-		(at 27.94 35.56 0)
+		(at 27.94 35.56 180)
 		(fields_autoplaced yes)
 		(effects
@@
 				(size 0.8 0.8)
 			)
-			(justify left bottom)
+			(justify right bottom)
 		)
 	)

Commit message: update
Parts:
- added R41: 3k3, Resistor_SMD:R_0402_1005Metric, symbol Device:R_Small
- added U42, U43: ASSR-1218, Package_SO:SO-4_4.4x4.3mm_P2.54mm, symbol Relay_SolidState:ASSR-1218
Connections:
- net +12V_RAW: now also U42.3; no longer FB4.2
- net -12V_RAW: now also U43.4; no longer FB3.2
- net GND: now also U42.2, U43.2
- new net: R41.1, U42.1, U43.1
- new net: FB3.2, U43.3
- new net: FB4.2, U42.4
- new net PWR_ANALOG_EN: R41.2
Other:
- moved on the sheet: C14, C17, C97, C98, FB3, FB4

Commit message: first ordered verrsion
Parts:
- removed D1: LED, LED_SMD:LED_0603_1608Metric, symbol Device:LED
- removed R4: 1k, Resistor_SMD:R_0402_1005Metric, symbol Device:R_Small
- removed R41: 3k3, Resistor_SMD:R_0402_1005Metric, symbol Device:R_Small
- removed U42, U43: ASSR-1218, Package_SO:SO-4_4.4x4.3mm_P2.54mm, symbol Relay_SolidState:ASSR-1218
Connections:
- net +12V_RAW: now also FB4.2
- net -12V_RAW: now also FB3.2
