File: outputs.kicad_sch (KiCad schematic)
At the start: 64 parts, among them J1 AudioJack2_SwitchT, J2 AudioJack2_SwitchT, J3 AudioJack2_SwitchT, J4 AudioJack2_SwitchT, J5 AudioJack2_SwitchT, J6 AudioJack2_SwitchT, J7 AudioJack2_SwitchT, J8 AudioJack2_SwitchT, U34 AD5734R, U35 AD5734R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

Commit message: rename symbol & footprint libs
Parts:
- J1, J2, J3, J4, J5, J6, J7, J8: footprint MyParts:Jack_3.5mm_QingPu_WQP-PJ398SM_Vertical_CircularHoles -> BMCV:Jack_3.5mm_QingPu_WQP-PJ398SM_Vertical_CircularHoles
- U34, U35: footprint MyParts:TSSOP-24-1EP_4.4x7.8mm_P0.65mm_EP3.2x5mm -> BMCV:TSSOP-24-1EP_4.4x7.8mm_P0.65mm_EP3.2x5mm; symbol MySymbols:AD57x4R -> BMCV:AD57x4R
Changed lines of the file:
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@@
 			)
 		)
-		(property "Footprint" "MyParts:Jack_3.5mm_QingPu_WQP-PJ398SM_Vertical_CircularHoles"
+		(property "Footprint" "BMCV:Jack_3.5mm_QingPu_WQP-PJ398SM_Vertical_CircularHoles"
 			(at 96.52 74.93 0)
 			(effects
@@
 			)
 		)
-		(property "Footprint" "MyParts:Jack_3.5mm_QingPu_WQP-PJ398SM_Vertical_CircularHoles"
+		(property "Footprint" "BMCV:Jack_3.5mm_QingPu_WQP-PJ398SM_Vertical_CircularHoles"
 			(at 96.52 25.4 0)
 			(effects
@@
 	)
 	(symbol
-		(lib_id "MySymbols:AD57x4R")
+		(lib_id "BMCV:AD57x4R")
 		(at 237.49 139.7 0)
 		(unit 1)
@@
 			)
 		)
-		(property "Footprint" "MyParts:TSSOP-24-1EP_4.4x7.8mm_P0.65mm_EP3.2x5mm"
+		(property "Footprint" "BMCV:TSSOP-24-1EP_4.4x7.8mm_P0.65mm_EP3.2x5mm"
 			(at 234.95 132.08 0)
 			(effects
@@
 			)
 		)
-		(property "Footprint" "MyParts:Jack_3.5mm_QingPu_WQP-PJ398SM_Vertical_CircularHoles"
+		(property "Footprint" "BMCV:Jack_3.5mm_QingPu_WQP-PJ398SM_Vertical_CircularHoles"
 			(at 214.63 76.2 0)
 			(effects
@@
 	)
 	(symbol
-		(lib_id "MySymbols:AD57x4R")
+		(lib_id "BMCV:AD57x4R")
 		(at 102.87 143.51 0)
 		(unit 1)
@@
 			)
 		)
-		(property "Footprint" "MyParts:TSSOP-24-1EP_4.4x7.8mm_P0.65mm_EP3.2x5mm"
+		(property "Footprint" "BMCV:TSSOP-24-1EP_4.4x7.8mm_P0.65mm_EP3.2x5mm"
 			(at 100.33 135.89 0)
 			(effects
@@
 			)
 		)
-		(property "Footprint" "MyParts:Jack_3.5mm_QingPu_WQP-PJ398SM_Vertical_CircularHoles"
+		(property "Footprint" "BMCV:Jack_3.5mm_QingPu_WQP-PJ398SM_Vertical_CircularHoles"
 			(at 96.52 49.53 0)
 			(effects
@@
 			)
 		)
-		(property "Footprint" "MyParts:Jack_3.5mm_QingPu_WQP-PJ398SM_Vertical_CircularHoles"
+		(property "Footprint" "BMCV:Jack_3.5mm_QingPu_WQP-PJ398SM_Vertical_CircularHoles"
 			(at 214.63 26.67 0)
 			(effects
@@
 			)
 		)
-		(property "Footprint" "MyParts:Jack_3.5mm_QingPu_WQP-PJ398SM_Vertical_CircularHoles"
+		(property "Footprint" "BMCV:Jack_3.5mm_QingPu_WQP-PJ398SM_Vertical_CircularHoles"
 			(at 214.63 101.6 0)
 			(effects
@@
 			)
 		)
-		(property "Footprint" "MyParts:Jack_3.5mm_QingPu_WQP-PJ398SM_Vertical_CircularHoles"
+		(property "Footprint" "BMCV:Jack_3.5mm_QingPu_WQP-PJ398SM_Vertical_CircularHoles"
 			(at 214.63 50.8 0)
 			(effects
@@
 			)
 		)
-		(property "Footprint" "MyParts:Jack_3.5mm_QingPu_WQP-PJ398SM_Vertical_CircularHoles"
+		(property "Footprint" "BMCV:Jack_3.5mm_QingPu_WQP-PJ398SM_Vertical_CircularHoles"
 			(at 96.52 100.33 0)
 			(effects

Commit message: Routing WIP
Connections:
- net OUT_BUFFERED_A1: now also R33.1; no longer R34.1
- net OUT_BUFFERED_A2: now also R38.1; no longer R37.1
- net OUT_BUFFERED_B1: now also R34.1; no longer R33.1
- net OUT_BUFFERED_B2: now also R37.1; no longer R38.1
- net OUT_BUFFERED_C1: now also R35.1; no longer R36.1
- net OUT_BUFFERED_C2: now also R40.1; no longer R39.1
- net OUT_BUFFERED_D1: now also R36.1; no longer R35.1
- net OUT_BUFFERED_D2: now also R39.1; no longer R40.1
- net at R21.1, U40.3 (+): now also R40.2; no longer R37.2
- net at R24.1, U40.12 (+): now also R38.2; no longer R40.2
- net at R16.1, U39.12 (+): now also R33.2; no longer R36.2
- net at R14.1, U39.5 (+): now also R36.2; no longer R34.2
- net at R22.1, U40.5 (+): now also R39.2; no longer R38.2
- net at R13.1, U39.3 (+): now also R35.2; no longer R33.2
- net at R23.1, U40.10 (+): now also R37.2; no longer R39.2
- net at R15.1, U39.10 (+): now also R34.2; no longer R35.2
- new net: J6.T, R27.2
- new net: J3.T, R17.2
- new net: J2.T, R19.2
- new net: J4.T, R20.2
- new net: J7.T, R25.2
- new net: J5.T, R26.2
- new net: J1.T, R18.2
- new net: J8.T, R28.2
- now unconnected: J1.TN, J2.TN, J3.TN, J4.TN, J5.TN, J6.TN, J7.TN, J8.TN
- no-connect marks 2 -> 10
Other:
- moved on the sheet: J1, J2, J3, J4, J5, J6, J7, J8, R33, R34, R35, R36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

Commit message: alpha
Parts:
- C22, C23, C24, C25, C48, C51, C54, C57, C73, C74: LCSC Part # (none) -> C14663
- C60, C63, C66, C68, C69, C70, C71, C72, C75, C76: footprint Capacitor_Tantalum_SMD:CP_EIA-3216-18_Kemet-A -> Capacitor_SMD:C_0805_2012Metric; LCSC Part # (none) -> C237493
- J1, J2, J3, J4, J5, J6, J7, J8: now not fitted
- R13, R14, R15, R16, R21, R22, R23, R24: footprint Resistor_SMD:R_0402_1005Metric -> Resistor_SMD:R_0603_1608Metric; LCSC Part # (none) -> C7250
- R17, R18, R19, R20, R25, R26, R27, R28: LCSC Part # (none) -> C22775
- R33, R34, R35, R36, R37, R38, R39, R40: LCSC Part # (none) -> C25076
- RV10, RV11, RV12, RV5, RV6, RV7, RV8, RV9: LCSC Part # (none) -> C210791
- U34, U35: LCSC Part # (none) -> C578284
- U39, U40: LCSC Part # (none) -> C529553

Commit message: update
Parts:
- J1, J2, J3, J4, J5, J6, J7, J8: now fitted
Changed lines of the file:
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@@
 		(in_bom yes)
 		(on_board yes)
-		(dnp yes)
+		(dnp no)
 		(property "Reference" "J3"
 			(at 101.6 23.4949 0)
@@
 		(in_bom yes)
 		(on_board yes)
-		(dnp yes)
+		(dnp no)
 		(property "Reference" "J2"
 			(at 102.87 75.438 0)
@@
 		(in_bom yes)
 		(on_board yes)
-		(dnp yes)
+		(dnp no)
 		(property "Reference" "J7"
 			(at 219.71 24.7649 0)
@@
 		(in_bom yes)
 		(on_board yes)
-		(dnp yes)
+		(dnp no)
 		(property "Reference" "J4"
 			(at 104.14 98.044 0)
@@
 		(in_bom yes)
 		(on_board yes)
-		(dnp yes)
+		(dnp no)
 		(property "Reference" "J6"
 			(at 219.71 74.2949 0)
@@
 		(in_bom yes)
 		(on_board yes)
-		(dnp yes)
+		(dnp no)
 		(property "Reference" "J5"
 			(at 219.71 48.8949 0)
@@
 		(in_bom yes)
 		(on_board yes)
-		(dnp yes)
+		(dnp no)
 		(property "Reference" "J8"
 			(at 219.71 99.6949 0)
@@
 		(in_bom yes)
 		(on_board yes)
-		(dnp yes)
+		(dnp no)
 		(property "Reference" "J1"
 			(at 103.378 47.244 0)

Commit message: update
Changed lines of the file:
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@@
 		(on_board yes)
 		(dnp no)
-		(fields_autoplaced yes)
 		(property "Reference" "#PWR043"
 			(at 252.73 160.02 0)
@@
 		)
 		(property "Value" "+3.3V"
-			(at 252.73 151.13 0)
+			(at 257.175 156.21 0)
 			(effects
 				(font
@@
 		(on_board yes)
 		(dnp no)
-		(fields_autoplaced yes)
 		(property "Reference" "#PWR064"
 			(at 118.11 163.83 0)
@@
 		)
 		(property "Value" "+3.3V"
-			(at 118.11 154.94 0)
-			(effects
-				(font
+			(at 121.92 160.02 0)
+			(effects
+				(font

Commit message: first ordered verrsion
Parts:
- RV10, RV11, RV12, RV5, RV6, RV7, RV8, RV9: value B72500D0160H060 -> SD12C-01FTG; footprint Resistor_SMD:R_0603_1608Metric -> Diode_SMD:D_SOD-323; symbol Device:Varistor -> Diode:SD12_SOD323; LCSC Part # C210791 -> C135970
- U34, U35: value AD5734R -> AD5754R; LCSC Part # C578284 -> C392906
Connections:
- net GND: now also RV10.1 (A1), RV11.1 (A1), RV12.1 (A1), RV5.1 (A1), RV6.1 (A1), RV7.1 (A1), RV8.1 (A1), RV9.1 (A1); no longer RV10.2, RV11.2, RV12.2, RV5.2, RV6.2, RV7.2, RV8.2, RV9.2
- net at R20.1, U39.13 (-), U39.14: now also RV8.2 (A2); no longer RV8.1
- net at R27.1, U40.8, U40.9 (-): now also RV11.2 (A2); no longer RV11.1
- net at R25.1, U40.1, U40.2 (-): now also RV9.2 (A2); no longer RV9.1
- net at R28.1, U40.13 (-), U40.14: now also RV12.2 (A2); no longer RV12.1
- net at R26.1, U40.6 (-), U40.7: now also RV10.2 (A2); no longer RV10.1
- net at R17.1, U39.1, U39.2 (-): now also RV5.2 (A2); no longer RV5.1
- net at R19.1, U39.8, U39.9 (-): now also RV7.2 (A2); no longer RV7.1
- net at R18.1, U39.6 (-), U39.7: now also RV6.2 (A2); no longer RV6.1

Commit message: kicad v9
Changed lines of the file:
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@@
 (kicad_sch
-	(version 20231120)
+	(version 20250114)
 	(generator "eeschema")
-	(generator_version "8.0")
+	(generator_version "9.0")
 	(paper "A4")
 	(junction
