File: inputs_cv.kicad_sch (KiCad schematic)
At the start: 37 parts, among them J10 AudioJack2_SwitchT, J11 AudioJack2_SwitchT, J12 AudioJack2_SwitchT, J9 AudioJack2_SwitchT, U33 AD7367-5, U38 OPA4171

Commit message: rename symbol & footprint libs
Parts:
- J10, J11, J12, J9: footprint MyParts:Jack_3.5mm_QingPu_WQP-PJ398SM_Vertical_CircularHoles -> BMCV:Jack_3.5mm_QingPu_WQP-PJ398SM_Vertical_CircularHoles
- U33: symbol MySymbols:AD736x -> BMCV:AD736x
Changed lines of the file:
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@@
 			)
 		)
-		(property "Footprint" "MyParts:Jack_3.5mm_QingPu_WQP-PJ398SM_Vertical_CircularHoles"
+		(property "Footprint" "BMCV:Jack_3.5mm_QingPu_WQP-PJ398SM_Vertical_CircularHoles"
 			(at 71.12 96.52 0)
 			(effects
@@
 			)
 		)
-		(property "Footprint" "MyParts:Jack_3.5mm_QingPu_WQP-PJ398SM_Vertical_CircularHoles"
+		(property "Footprint" "BMCV:Jack_3.5mm_QingPu_WQP-PJ398SM_Vertical_CircularHoles"
 			(at 71.12 71.12 0)
 			(effects
@@
 			)
 		)
-		(property "Footprint" "MyParts:Jack_3.5mm_QingPu_WQP-PJ398SM_Vertical_CircularHoles"
+		(property "Footprint" "BMCV:Jack_3.5mm_QingPu_WQP-PJ398SM_Vertical_CircularHoles"
 			(at 71.12 121.92 0)
 			(effects
@@
 	)
 	(symbol
-		(lib_id "MySymbols:AD736x")
+		(lib_id "BMCV:AD736x")
 		(at 218.44 78.74 0)
 		(unit 1)
@@
 			)
 		)
-		(property "Footprint" "MyParts:Jack_3.5mm_QingPu_WQP-PJ398SM_Vertical_CircularHoles"
+		(property "Footprint" "BMCV:Jack_3.5mm_QingPu_WQP-PJ398SM_Vertical_CircularHoles"
 			(at 71.12 46.99 0)
 			(effects

Commit message: clea up project
Connections:
- net at J9.T, J9.TN: now also R31.1; no longer R30.1
- net at J10.T, J10.TN: now also R30.1; no longer R31.1
- net at U38.1, U38.2 (-): now also R9.1; no longer R6.1
- net at J12.T, J12.TN: now also R29.1; no longer R32.1
- net at U38.13 (-), U38.14: now also R7.1; no longer R9.1
- net at U38.6 (-), U38.7: now also R8.1; no longer R7.1
- net at U38.8, U38.9 (-): now also R6.1; no longer R8.1
- net at J11.T, J11.TN: now also R32.1; no longer R29.1
Other:
- moved on the sheet: J10, J11, J12, J9, R6, R7, R8, R9

Commit message: Routing WIP
Connections:
- net IN_BUFFERED_A1: now also R7.2; no longer R6.2
- net IN_BUFFERED_A2: now also R6.2; no longer R7.2
- net IN_BUFFERED_B1: now also R9.2; no longer R8.2
- net IN_BUFFERED_B2: now also R8.2; no longer R9.2
- new net: J12.T, R30.1
- new net: J11.T, R31.1
- new net: J9.T, R32.1
- new net: J10.T, R29.1
- now unconnected: J10.TN, J11.TN, J12.TN, J9.TN
- no-connect marks 0 -> 4
Other:
- moved on the sheet: J10, J11, J12, J9

Commit message: alpha
Parts:
- C20, C21, C87, C89: LCSC Part # (none) -> C14663
- C77, C79, C80, C81, C88, C90: footprint Capacitor_Tantalum_SMD:CP_EIA-3216-18_Kemet-A -> Capacitor_SMD:C_0805_2012Metric; LCSC Part # (none) -> C237493
- C78, C82, C83: LCSC Part # (none) -> C307331
- C85, C86: LCSC Part # (none) -> C5143539
- J10, J11, J12, J9: now not fitted
- R10, R11, R12, R5: footprint Resistor_SMD:R_0402_1005Metric -> Resistor_SMD:R_0603_1608Metric; LCSC Part # (none) -> C7250
- R29, R30, R31, R32: LCSC Part # (none) -> C22775
- R6, R7, R8, R9: LCSC Part # (none) -> C25076
- RV1, RV2, RV3, RV4: LCSC Part # (none) -> C210791
- U33: LCSC Part # (none) -> C650862
- U38: LCSC Part # (none) -> C529553

Commit message: update
Parts:
- J10, J11, J12, J9: now fitted
Changed lines of the file:
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@@
 		(in_bom yes)
 		(on_board yes)
-		(dnp yes)
+		(dnp no)
 		(property "Reference" "J10"
 			(at 70.485 55.88 0)
@@
 		(in_bom yes)
 		(on_board yes)
-		(dnp yes)
+		(dnp no)
 		(property "Reference" "J9"
 			(at 70.485 130.81 0)
@@
 		(in_bom yes)
 		(on_board yes)
-		(dnp yes)
+		(dnp no)
 		(property "Reference" "J12"
 			(at 70.485 80.01 0)
@@
 		(in_bom yes)
 		(on_board yes)
-		(dnp yes)
+		(dnp no)
 		(property "Reference" "J11"
 			(at 70.485 105.41 0)

Commit message: first ordered verrsion
Parts:
- RV1, RV2, RV3, RV4: value B72500D0160H060 -> SD12C-01FTG; footprint Resistor_SMD:R_0603_1608Metric -> Diode_SMD:D_SOD-323; symbol Device:Varistor -> Diode:SD12_SOD323; LCSC Part # C210791 -> C135970
Connections:
- net GND: now also RV1.1 (A1), RV2.1 (A1), RV3.1 (A1), RV4.1 (A1); no longer RV1.2, RV2.2, RV3.2, RV4.2
- net at R10.1, R30.2, U38.5 (+): now also RV2.2 (A2); no longer RV2.1
- net at R11.1, R31.2, U38.10 (+): now also RV3.2 (A2); no longer RV3.1
- net at R29.2, R5.1, U38.3 (+): now also RV1.2 (A2); no longer RV1.1
- net at R12.1, R32.2, U38.12 (+): now also RV4.2 (A2); no longer RV4.1

Commit message: kicad v9
Changed lines of the file:
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@@
 (kicad_sch
-	(version 20231120)
+	(version 20250114)
 	(generator "eeschema")
-	(generator_version "8.0")
+	(generator_version "9.0")
 	(paper "A4")
 	(junction
@@
 	(label "DCAPA"
 		(at 182.88 138.43 180)
-		(fields_autoplaced yes)
 		(effects
 			(font
@@
 	(label "DCAPA"
 		(at 198.12 86.36 0)
-		(fields_autoplaced yes)
 		(effects
 			(font
@@
 	(label "DCAPB"
 		(at 193.04 138.43 0)
-		(fields_autoplaced yes)
 		(effects
 			(font
@@
 	(label "DCAPB"
 		(at 238.76 86.36 180)
-		(fields_autoplaced yes)
 		(effects
 			(font

Commit message: pcb changes
Parts:
- added C100, C101, C102, C103: 1nF, Capacitor_SMD:C_0402_1005Metric, symbol Device:C_Small
- R10, R11, R12, R5: value 10M -> 1M; LCSC Part # C7250 -> C22935
Connections:
- net GND: now also C100.1, C101.1, C102.1, C103.1
- net at R10.1, R30.2, RV2.2 (A2)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: now also C101.2
- net at R11.1, R31.2, RV3.2 (A2)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: now also C102.2
- net at R29.2, R5.1, RV1.2 (A2)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: now also C100.2
- net at R12.1, R32.2, RV4.2 (A2)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: now also C103.2
