File: encoders.kicad_sch (KiCad schematic)
At the start: 109 parts, among them U1 PEL12T-4225S-S1024, U10 WS2811F, U11 WS2811F, U12 WS2811F, U13 WS2811F, U14 WS2811F, U15 WS2811F, U16 WS2811F, U2 PEL12T-4225S-S1024, U3 PEL12T-4225S-S1024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

Commit message: add test firwmware
Connections:
- net MCP_5V_BTN_INT: now reaches U30.20 (INTA)
- net MCP_5V_ENCINT_A: no longer names the net of U31.19 (INTB)
- net MCP_5V_ENCINT_B renamed MCP_5V_ENC_INT
Changed lines of the file:
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@@
 	)
 	(no_connect
-		(at 240.03 49.53)
-	)
-	(no_connect
 		(at 182.88 38.1)
 	)
@@
 		(at 133.35 115.57)
 	)
+	(no_connect
+		(at 240.03 123.19)
+	)
 	(wire
 		(pts
@@
 	(wire
 		(pts
+			(xy 234.95 125.73) (xy 240.03 125.73)
+		)
+		(stroke
+			(width 0)
+			(type default)
+		)
+	)
+	(wire
+		(pts
 			(xy 78.74 123.19) (xy 86.36 123.19)
 		)
@@
 	(wire
 		(pts
-			(xy 234.95 123.19) (xy 240.03 123.19)
-		)
-		(stroke
-			(width 0)
-			(type default)
-		)
-	)
-	(wire
-		(pts
 			(xy 151.13 33.02) (xy 151.13 34.29)
 		)
@@
 	(wire
 		(pts
-			(xy 234.95 125.73) (xy 240.03 125.73)
+			(xy 234.95 49.53) (xy 240.03 49.53)
 		)
 		(stroke
@@
 		)
 	)
-	(global_label "MCP_5V_ENCINT_B"
+	(global_label "MCP_5V_BTN_INT"
 		(shape input)
-		(at 234.95 125.73 180)
+		(at 234.95 49.53 180)
 		(fields_autoplaced yes)
 		(effects
@@
 		)
 		(property "Intersheetrefs" "${INTERSHEET_REFS}"
-			(at 214.8501 125.73 0)
+			(at 216.3015 49.53 0)
 			(effects
 				(font
@@
 		)
 	)
+	(global_label "MCP_5V_ENC_INT"
+		(shape input)
+		(at 234.95 125.73 180)
+		(fields_autoplaced yes)
+		(effects
+			(font
+				(size 1.27 1.27)
+			)
+			(justify right)
+		)
+		(property "Intersheetrefs" "${INTERSHEET_REFS}"
+			(at 216.1201 125.73 0)
+			(effects
+				(font
+					(size 1.27 1.27)
+				)
+				(justify right)
+				(hide yes)
+			)
+		)
+	)
 	(global_label "ENC_6_SW"
 		(shape input)
@@
 				(hide yes)
 			)
-		)
-	)
-	(global_label "MCP_5V_ENCINT_A"
-		(shape input)
-		(at 234.95 123.19 180)
-		(fields_autoplaced yes)
-		(effects
-			(font
-				(size 1.27 1.27)
-			)
-			(justify right)
-		)
-		(property "Intersheetrefs" "${INTERSHEET_REFS}"
-			(at 215.0315 123.19 0)
-			(effects
-				(font
-					(size 1.27 1.27)
-				)
-				(justify right)
-				(hide yes)
-			)
