File: BMCV.kicad_sch (KiCad schematic)
At the start: 42 parts, among them J13 EXTRA_PIN_1, J14 USB_C_Receptacle_USB2.0_14P, SW14 FN1, SW15 FN2/Boot, SW16 FN3, U32 TXS0108EPW, U36 STM32G474CETx, U37 MB85RS64PNF-G-JNERE1, U42 74AHCT1G125, Y1 38.4MHz 10pF

Commit message: v1
Parts:
- J13: now not fitted; now left out of the parts list
- U42: LCSC Part # (none) -> C151417
Connections:
- net at RV13.2: now also R158.2
- net at RV13.5: no longer R158.2
Changed lines of the file:
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@@
 	)
 	(no_connect
-		(at 29.21 189.865)
+		(at 41.91 189.865)
 	)
 	(wire
@@
 	(wire
 		(pts
-			(xy 41.91 186.69) (xy 41.91 189.865)
-		)
-		(stroke
-			(width 0)
-			(type default)
-		)
-	)
-	(wire
-		(pts
 			(xy 120.015 78.74) (xy 120.015 76.835)
 		)
@@
 	(wire
 		(pts
+			(xy 29.21 186.69) (xy 29.21 189.865)
+		)
+		(stroke
+			(width 0)
+			(type default)
+		)
+	)
+	(wire
+		(pts
 			(xy 140.97 187.96) (xy 140.97 193.04)
 		)
@@
 	(wire
 		(pts
-			(xy 43.18 186.69) (xy 41.91 186.69)
-		)
-		(stroke
-			(width 0)
-			(type default)
-		)
-	)
-	(wire
-		(pts
 			(xy 364.49 226.695) (xy 367.03 226.695)
 		)
@@
 	(wire
 		(pts
+			(xy 29.21 186.69) (xy 43.18 186.69)
+		)
+		(stroke
+			(width 0)
+			(type default)
+		)
+	)
+	(wire
+		(pts
 			(xy 59.69 265.43) (xy 59.69 270.51)
 		)
@@
 			)
 		)
+		(property "LCSC Part #" "C151417"
+			(at 236.22 227.33 0)
+			(effects
+				(font
+					(size 1.27 1.27)
+				)
+				(hide yes)
+			)
+		)
 		(property "Height" ""
 			(at 236.22 227.33 0)
@@
 		(unit 1)
 		(exclude_from_sim no)
-		(in_bom yes)
+		(in_bom no)
 		(on_board yes)
-		(dnp no)
+		(dnp yes)
 		(fields_autoplaced yes)
 		(property "Reference" "J13"
